File: pcb/lever.kicad_pcb (KiCad board)
At the start: 2 copper layers, 40 x 28.6 mm, 12 parts, among them J1 RJ45_pyControl, J2 Conn_01x02, J3 Conn_01x03, U1 ATtiny84-20SSU, X1 AVR_ISP

Commit message: pcb v1.1
Parts:
- moved X1 3.17 mm to (125.1, 81.3)
- moved J2 1.02 mm to (132.7, 74.7)
Routing:
- net Net-(U1-Pad4): track 24.7 -> 17.3 mm
- net Net-(J3-Pad1): track 31.4 -> 28.3 mm, vias 1 -> 0
- net /DIO_C: track 23.1 -> 25.9 mm
- net /DIO_B: track 29.1 -> 26.8 mm
- net /Vcc: track 52.2 -> 50.2 mm
- net Net-(U1-Pad7): track 20.5 -> 18.7 mm
- net /DIO_A: track 32.8 -> 31.4 mm
Other:
- board text added: "Lever v1.1"
- board text removed: "Lever v1.0"
