File: pcb/lever.sch (KiCad schematic (older format))
At the start: 12 parts, among them J1 RJ45_pyControl, J2 Conn_01x02, J3 Conn_01x03, U1 ATtiny84-20SSU, X1 AVR_ISP

Commit message: PCB bom and rendering updates
Parts:
- C1: value 0.1µF -> 0.1 µF
- D1: value LED -> Red
- J1: value RJ45_pyControl -> 0855135013
- R1: value 10KΩ -> 20KΩ
- U1: value ATtiny84-20SSU -> ATTINY24A-SSUR; Description ATtiny 84 MCU -> ATtiny 24 MCU
- X1: value AVR_ISP -> 75869-331LF
Changed lines of the file:
@@
 	5400 3200 5400 3550
 Wire Wire Line
-	7700 3550 7700 5500
+	8050 3550 8050 5500
 $Comp
 L asl_symbols:AVR_ISP X1
@@
 P 5250 5000
 F 0 "X1" H 5250 5325 50  0000 C CNN
-F 1 "AVR_ISP" H 5250 5234 50  0000 C CNN
+F 1 "75869-331LF" H 5250 5234 50  0000 C CNN
 F 2 "asl_footprints:AVR_ISP" H 5100 4950 50  0001 C CNN
 F 3 "https://www.digikey.com/products/en?keywords=609-5122-ND" H 5100 4950 50  0001 C CNN
@@
 P 5650 2750
 F 0 "J1" H 5682 3325 50  0000 C CNN
-F 1 "RJ45_pyControl" H 5682 3234 50  0000 C CNN
+F 1 "0855135013" H 5682 3234 50  0000 C CNN
 F 2 "asl_footprints:RJ45_SMD_Vertical" H 5700 2200 50  0001 C CNN
 F 3 "https://www.digikey.com/products/en?keywords=WM3553CT-ND" V 5550 2725 50  0001 C CNN
@@
 P 4500 4450
 F 0 "D1" H 4493 4666 50  0000 C CNN
-F 1 "LED" H 4493 4575 50  0000 C CNN
+F 1 "Red" H 4493 4575 50  0000 C CNN
 F 2 "LED_SMD:LED_0603_1608Metric_Pad1.05x0.95mm_HandSolder" H 4500 4450 50  0001 C CNN
-F 3 "~" H 4500 4450 50  0001 C CNN
+F 3 "https://www.digikey.com/products/en?keywords=160-1447-1-ND" H 4500 4450 50  0001 C CNN
 F 4 "Indicator LED" H 4500 4450 50  0001 C CNN "Description"
 	1    4500 4450
@@
 	4900 5500 6850 5500
 Wire Wire Line
-	7700 5500 6850 5500
+	8050 5500 6850 5500
 Wire Wire Line
 	6850 3650 6850 3700
@@
 P 6850 4600
 F 0 "U1" H 6320 4646 50  0000 R CNN
-F 1 "ATtiny84-20SSU" H 6320 4555 50  0000 R CNN
+F 1 "ATTINY24A-SSUR" H 6320 4555 50  0000 R CNN
 F 2 "Package_SO:SOIC-14_3.9x8.7mm_P1.27mm" H 6850 4600 50  0001 C CIN
-F 3 "http://ww1.microchip.com/downloads/en/DeviceDoc/doc8006.pdf" H 6850 4600 50  0001 C CNN
-F 4 "ATtiny 84 MCU" H 6850 4600 50  0001 C CNN "Description"
+F 3 "https://www.digikey.com/products/en?keywords=ATTINY24A-SSURCT-ND" H 6850 4600 50  0001 C CNN
+F 4 "ATtiny 24 MCU" H 6850 4600 50  0001 C CNN "Description"
 	1    6850 4600
 	-1   0    0    -1
@@
 P 4250 4950
 F 0 "R1" H 4182 4904 50  0000 R CNN
-F 1 "10KΩ" H 4182 4995 50  0000 R CNN
+F 1 "20KΩ" H 4182 4995 50  0000 R CNN
 F 2 "Resistor_SMD:R_0603_1608Metric_Pad1.05x0.95mm_HandSolder" V 4290 4940 50  0001 C CNN
 F 3 "~" H 4250 4950 50  0001 C CNN
@@
 P 7000 3650
 F 0 "C1" V 6748 3650 50  0000 C CNN
-F 1 "0.1µF" V 6839 3650 50  0000 C CNN
+F 1 "0.1 µF" V 6839 3650 50  0000 C CNN
 F 2 "Capacitor_SMD:C_0603_1608Metric_Pad1.05x0.95mm_HandSolder" H 7038 3500 50  0001 C CNN
-F 3 "~" H 7000 3650 50  0001 C CNN
+F 3 "https://www.digikey.com/products/en?keywords=1276-1258-1-ND" H 7000 3650 50  0001 C CNN
 	1    7000 3650
 	0    1    1    0
@@
 Connection ~ 7150 3550
 Wire Wire Line
-	7150 3550 7700 3550
+	7150 3550 8050 3550
 $Comp
 L Device:C C2
